File: GB-BRK-M/GB-BRK-M.sch (EAGLE design)
At the start: 2 parts

Commit message: GB-BRK-M v2.1
Parts:
- added C1: 0.1uF, SparkFun-Capacitors:CAP1206
- JP1: device pinhead:PINHD-2X16 -> pinhead+:PINHD-2X16SMT
Connections:
- removed net MREQ: JP1.10, U$2./MREQ
- removed net RD: JP1.8, U$2./RD
- removed net RST: JP1.28, U$2./RST
- removed net WR: JP1.6, U$2./WR
- new net !CS: JP1.10, U$2.!CS
- new net !RD: JP1.8, U$2.!RD
- new net !RST: JP1.28, U$2.!RST
- new net !WR: JP1.6, U$2.!WR
- net GND: now also C1.2
- net VCC: now also C1.1
Other:
- note removed: "gekkio"
- note removed: "http://gekkio.fi"
- note removed: "v1.0"
- moved on the sheet: JP1, U$2
