File: GB-BRK-M/GB-BRK-M.kicad_pcb (KiCad board)
At the start: 2 copper layers, 51.4 x 61 mm, 15 parts, among them J1 CONN_02X16, J2 Conn_GameBoy_Cartridge

Commit message: GB-BRK-M v3.1
Parts:
- C1: footprint Capacitors_SMD:C_0805 -> Capacitor_SMD:C_0805_2012Metric
- D1, D2, D3: value LED -> LED_Y; footprint LEDs:LED_0603 -> LED_SMD:LED_0603_1608Metric
- D4, D5: value LED -> LED_R; footprint LEDs:LED_0603 -> LED_SMD:LED_0603_1608Metric
- J1: footprint Pin_Headers:Pin_Header_Straight_2x16_Pitch2.54mm_SMD -> Connector_PinHeader_2.54mm:PinHeader_2x16_P2.54mm_Vertical_SMD
- R1, R2, R3, R4, R5: footprint Resistors_SMD:R_0603 -> Resistor_SMD:R_0603_1608Metric
Other:
- board text added: "GB-BRK-M v3.1 https://gekkio.fi"
- board text removed: "GB-BRK-M v3.0 https://gekkio.fi"
