File: GB-BRK-CART/GB-BRK-CART.sch (KiCad schematic (older format))
At the start: 7 parts, among them J1 Conn_02x16_Odd_Even, J2 GameBoy_Cartridge

Commit message: Minor fixes + add schematic
Parts:
- J1: MPN 15-91-0400 -> 15-91-0800; SPN 538-15-91-0400 -> 538-15-91-0800
- R1: value 330 -> 3.3k; MPN CRCW0603330RFKEA -> CRCW06033K30JNEB; Rating 1/10W 1% -> 1/10W 5%; SPN 71-CRCW0603-330-E3 -> 71-CRCW06033K30JNEB
Other:
- note added: "Optional"
Changed lines of the file:
@@
 F 3 "" H 5600 3200 50  0001 C CNN
 F 4 "Molex" H 5700 4150 50  0001 C CNN "MFR"
-F 5 "15-91-0400" H 5800 4250 50  0001 C CNN "MPN"
+F 5 "15-91-0800" H 5800 4250 50  0001 C CNN "MPN"
 F 6 "Mouser" H 5900 4350 50  0001 C CNN "SPR"
-F 7 "538-15-91-0400" H 6000 4450 50  0001 C CNN "SPN"
+F 7 "538-15-91-0800" H 6000 4450 50  0001 C CNN "SPN"
 F 8 "" H 0   0   50  0001 C CNN "Rating"
 	1    5600 3200
@@
 L Device:R R1
 U 1 1 5910CAE9
-P 8250 3000
-F 0 "R1" V 8330 3000 50  0000 C CNN
-F 1 "330" V 8250 3000 50  0000 C CNN
-F 2 "Resistor_SMD:R_0603_1608Metric" V 8180 3000 50  0001 C CNN
-F 3 "" H 8250 3000 50  0001 C CNN
-F 4 "Vishay" H 0   -1250 50  0001 C CNN "MFR"
-F 5 "CRCW0603330RFKEA" H 0   -1250 50  0001 C CNN "MPN"
-F 6 "Mouser" H 0   -1250 50  0001 C CNN "SPR"
-F 7 "71-CRCW0603-330-E3" H 0   -1250 50  0001 C CNN "SPN"
-F 8 "1/10W 1%" V 8250 3000 60  0001 C CNN "Rating"
-	1    8250 3000
+P 9650 4100
+F 0 "R1" V 9730 4100 50  0000 C CNN
+F 1 "3.3k" V 9650 4100 50  0000 C CNN
+F 2 "Resistor_SMD:R_0603_1608Metric" V 9580 4100 50  0001 C CNN
+F 3 "" H 9650 4100 50  0001 C CNN
+F 4 "Vishay" H 1400 -150 50  0001 C CNN "MFR"
+F 5 "CRCW06033K30JNEB" H 1400 -150 50  0001 C CNN "MPN"
+F 6 "Mouser" H 1400 -150 50  0001 C CNN "SPR"
+F 7 "71-CRCW06033K30JNEB" H 1400 -150 50  0001 C CNN "SPN"
+F 8 "1/10W 5%" V 9650 4100 60  0001 C CNN "Rating"
+	1    9650 4100
 	0    1    1    0
 $EndComp
@@
 L Device:LED D1
 U 1 1 5910CC2A
-P 7950 3000
-F 0 "D1" H 7950 3100 50  0000 C CNN
-F 1 "LED_R" H 8000 2900 50  0000 C CNN
-F 2 "LED_SMD:LED_0603_1608Metric" H 7950 3000 50  0001 C CNN
-F 3 "" H 7950 3000 50  0001 C CNN
-F 4 "Wurth Electronics" H 0   -1250 50  0001 C CNN "MFR"
-F 5 "150060SS75000" H 0   -1250 50  0001 C CNN "MPN"
-F 6 "Mouser" H 0   -1250 50  0001 C CNN "SPR"
-F 7 "710-150060SS75000" H 0   -1250 50  0001 C CNN "SPN"
-F 8 "" H 0   0   50  0001 C CNN "Rating"
-	1    7950 3000
+P 9350 4100
+F 0 "D1" H 9350 4200 50  0000 C CNN
+F 1 "LED_R" H 9400 4000 50  0000 C CNN
+F 2 "LED_SMD:LED_0603_1608Metric" H 9350 4100 50  0001 C CNN
+F 3 "" H 9350 4100 50  0001 C CNN
+F 4 "Wurth Electronics" H 1400 -150 50  0001 C CNN "MFR"
+F 5 "150060SS75000" H 1400 -150 50  0001 C CNN "MPN"
+F 6 "Mouser" H 1400 -150 50  0001 C CNN "SPR"
+F 7 "710-150060SS75000" H 1400 -150 50  0001 C CNN "SPN"
+F 8 "" H 1400 1100 50  0001 C CNN "Rating"
+	1    9350 4100
 	1    0    0    -1
 $EndComp
@@
 L power:GND #PWR07
 U 1 1 5963F136
-P 7600 3000
-F 0 "#PWR07" H 7600 2750 50  0001 C CNN
-F 1 "GND" H 7600 2850 50  0000 C CNN
-F 2 "" H 7600 3000 50  0001 C CNN
-F 3 "" H 7600 3000 50  0001 C CNN
-	1    7600 3000
+P 9000 4100
+F 0 "#PWR07" H 9000 3850 50  0001 C CNN
+F 1 "GND" H 9000 3950 50  0000 C CNN
+F 2 "" H 9000 4100 50  0001 C CNN
+F 3 "" H 9000 4100 50  0001 C CNN
+	1    9000 4100
 	1    0    0    -1
 $EndComp
@@
 	5200 4000 5200 5100
 Wire Wire Line
-	8500 3000 8400 3000
-Wire Wire Line
-	7800 3000 7600 3000
+	9900 4100 9800 4100
+Wire Wire Line
+	9200 4100 9000 4100
 Connection ~ 5200 5100
 Wire Wire Line
@@
 L power:+5V #PWR05
 U 1 1 5AE67D6A
-P 8500 3000
-F 0 "#PWR05" H 8500 2850 50  0001 C CNN
-F 1 "+5V" H 8500 3140 50  0000 C CNN
-F 2 "" H 8500 3000 50  0001 C CNN
-F 3 "" H 8500 3000 50  0001 C CNN
-	1    8500 3000
+P 9900 4100
+F 0 "#PWR05" H 9900 3950 50  0001 C CNN
+F 1 "+5V" H 9900 4240 50  0000 C CNN
+F 2 "" H 9900 4100 50  0001 C CNN
+F 3 "" H 9900 4100 50  0001 C CNN
+	1    9900 4100
 	1    0    0    -1
 $EndComp
@@
 	9200 3500 9600 3500
 Connection ~ 9600 3500
+Wire Notes Line
+	8800 2900 8800 4400
+Wire Notes Line
+	8800 4400 10100 4400
+Wire Notes Line
+	10100 4400 10100 2900
+Wire Notes Line
+	10100 2900 8800 2900
+Text Notes 8800 2900 0    50   ~ 0
+Optional
 $EndSCHEMATC

Commit message: BOM + docs
Parts:
- C1: Rating 50V X7R -> 16V X5R
- J2: value GameBoy_Cartridge -> DNF
- MK1, MK2: value Mounting_Hole -> DNF
Changed lines of the file:
@@
 P 7600 1300
 F 0 "MK1" H 7600 1500 50  0000 C CNN
-F 1 "Mounting_Hole" H 7600 1425 50  0000 C CNN
+F 1 "DNF" H 7600 1425 50  0000 C CNN
 F 2 "Gekkio_MountingHole:MountingHole_7.2mm" H 7600 1300 50  0001 C CNN
 F 3 "" H 7600 1300 50  0001 C CNN
@@
 P 8300 1300
 F 0 "MK2" H 8300 1500 50  0000 C CNN
-F 1 "Mounting_Hole" H 8300 1425 50  0000 C CNN
+F 1 "DNF" H 8300 1425 50  0000 C CNN
 F 2 "Gekkio_MountingHole:MountingHole_2.3mm" H 8300 1300 50  0001 C CNN
 F 3 "" H 8300 1300 50  0001 C CNN
@@
 P 6500 3600
 F 0 "J2" H 6730 3650 50  0000 L CNN
-F 1 "GameBoy_Cartridge" H 6730 3559 50  0000 L CNN
+F 1 "DNF" H 6730 3559 50  0000 L CNN
 F 2 "Gekkio_Connector_PCBEdge:GameBoy_Cartridge_1x32_P1.50mm_Edge" H 6400 1800 50  0001 C CNN
 F 3 "" H 6400 3600 50  0001 L CNN
@@
 F 6 "Mouser" H 200 50  50  0001 C CNN "SPR"
 F 7 "581-06035C104KAT4A" H 200 50  50  0001 C CNN "SPN"
-F 8 "50V X7R" H 9600 3350 60  0001 C CNN "Rating"
+F 8 "16V X5R" H 9600 3350 60  0001 C CNN "Rating"
 	1    9600 3350
 	1    0    0    -1
