File: GB-BRK-CART/GB-BRK-CART.kicad_pcb (KiCad board)
At the start: 2 copper layers, 51.4 x 61 mm, 7 parts, among them J1 Conn_02x16_Odd_Even, J2 GameBoy_Cartridge

Commit message: Minor fixes + add schematic
Other:
- board text added: "PCB size: 51.4x61 mm"
Changed lines of the file:
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@@
-(kicad_pcb (version 20171130) (host pcbnew 5.0.0-rc2-unknown-01c2d93~65~ubuntu18.04.1)
+(kicad_pcb (version 20171130) (host pcbnew 5.0.0-rc3-unknown-101b68b~65~ubuntu18.04.1)
   (general
-    (thickness 1.6)
-    (drawings 49)
+    (thickness 0.8)
+    (drawings 50)
     (tracks 343)
     (zones 0)
@@
     )
   )
-  (gr_text "PCB thickness: 0.8 mm" (at 141.3 105.5) (layer F.Fab)
-    (effects (font (size 1.5 1.5) (thickness 0.3)))
+  (gr_text "PCB size: 51.4x61 mm" (at 128 105) (layer F.Fab)
+    (effects (font (size 1.5 1.5) (thickness 0.3)) (justify left))
+  )
+  (gr_text "PCB thickness: 0.8 mm" (at 128 108) (layer F.Fab)
+    (effects (font (size 1.5 1.5) (thickness 0.3)) (justify left))
   )
   (dimension 52.4 (width 0.3) (layer F.Fab)

Commit message: More details and fixes
Other:
- board text added: "PCB size: 51.4x61mm PCB thickness: 0.8mm"
- board text removed: "PCB size: 51.4x61 mm"
- board text removed: "PCB thickness: 0.8 mm"
Changed lines of the file:
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@@
   (general
     (thickness 0.8)
-    (drawings 50)
+    (drawings 49)
     (tracks 343)
     (zones 0)
@@
     )
   )
-  (gr_text "PCB size: 51.4x61 mm" (at 128 105) (layer F.Fab)
+  (gr_text "PCB size: 51.4x61mm\nPCB thickness: 0.8mm" (at 127 104) (layer F.Fab)
     (effects (font (size 1.5 1.5) (thickness 0.3)) (justify left))
   )
-  (gr_text "PCB thickness: 0.8 mm" (at 128 108) (layer F.Fab)
-    (effects (font (size 1.5 1.5) (thickness 0.3)) (justify left))
-  )

Commit message: BOM + docs
Parts:
- J2: value GameBoy_Cartridge -> DNF
- MK1, MK2: value Mounting_Hole -> DNF
- R1: value 330 -> 3.3k
Changed lines of the file:
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@@
       (effects (font (size 1 1) (thickness 0.15)))
     )
-    (fp_text value Mounting_Hole (at 0 2.2) (layer F.Fab) hide
+    (fp_text value DNF (at 0 2.2) (layer F.Fab) hide
       (effects (font (size 1 1) (thickness 0.15)))
     )
@@
       (effects (font (size 1 1) (thickness 0.15)))
     )
-    (fp_text value Mounting_Hole (at 0 5) (layer F.Fab) hide
+    (fp_text value DNF (at 0 5) (layer F.Fab) hide
       (effects (font (size 1 1) (thickness 0.15)))
     )
@@
       (effects (font (size 1 1) (thickness 0.15)))
     )
-    (fp_text value 330 (at -4 -0.1 180) (layer F.Fab)
+    (fp_text value 3.3k (at -4 -0.1 180) (layer F.Fab)
       (effects (font (size 1 1) (thickness 0.15)))
     )
@@
       (effects (font (size 1 1) (thickness 0.15)))
     )
-    (fp_text value GameBoy_Cartridge (at 0 -8) (layer F.Fab) hide
-      (effects (font (size 1 1) (thickness 0.15)))
-    )
+    (fp_text value DNF (at 0 -8) (layer F.Fab) hide
+      (effects (font (size 1 1) (thickness 0.15)))
+    )

Commit message: Update PCB size and thickness recommendations
Other:
- board text added: "PCB size: 51.4x61mm PCB thickness: 1.0mm"
- board text removed: "PCB size: 51.4x61mm PCB thickness: 0.8mm"
Changed lines of the file:
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@@
-(kicad_pcb (version 20171130) (host pcbnew 5.0.0-rc3-unknown-101b68b~65~ubuntu18.04.1)
+(kicad_pcb (version 20171130) (host pcbnew 5.0.2-bee76a0~70~ubuntu18.10.1)
   (general
-    (thickness 0.8)
+    (thickness 1)
     (drawings 49)
     (tracks 343)
@@
     )
   )
-  (gr_text "PCB size: 51.4x61mm\nPCB thickness: 0.8mm" (at 127 104) (layer F.Fab)
+  (gr_text "PCB size: 51.4x61mm\nPCB thickness: 1.0mm" (at 127 104) (layer F.Fab)
     (effects (font (size 1.5 1.5) (thickness 0.3)) (justify left))
   )

Commit message: Adjust solder mask clearances, regenerate gerbers
Other:
- rule pad_to_mask_clearance: 0.2 -> 0
Changed lines of the file:
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@@
     (pad_size 2.25 2.25)
     (pad_drill 2.25)
-    (pad_to_mask_clearance 0.2)
+    (pad_to_mask_clearance 0)
     (solder_mask_min_width 0.2)
     (aux_axis_origin 0 0)
@@
       (usegerberattributes false)
       (usegerberadvancedattributes false)
-      (creategerberjobfile false)
+      (creategerberjobfile true)
       (excludeedgelayer false)
       (linewidth 0.100000)

Commit message: Upgrade most projects to KiCad 6
Connections:
- net /~CS renamed /~{CS}
- net /~RD renamed /~{RD}
- net /~RES renamed /~{RES}
- net /~WR renamed /~{WR}
Other:
- net class Default removed
- net class Power removed
- board text added: "~{CS}"
- board text added: "~{RD}"
- board text added: "~{RES}"
- board text added: "~{WR}"
- board text removed: "~CS"
- board text removed: "~RD"
- board text removed: "~RES"
- board text removed: "~WR"
