File: GB-LIVE32/GB-LIVE32.sch (KiCad schematic (older format))
At the start: 39 parts, among them J1 Conn_01x05, U1 MCP1703A-3302_SOT89, U2 PIC18LF45K50_QFP, U3 IS61LV256AL-10T

Commit message: BOM + docs
Parts:
- C1, C3: MFR (none) -> Taiyo Yuden; MPN (none) -> EMK212BJ475MD-T; Rating (none) -> 16V X5R; SPN (none) -> 963-EMK212BJ475MD-T; SPR (none) -> Mouser
- C2: MFR (none) -> KEMET; MPN (none) -> C0603C474K4PACTU; Rating (none) -> 16V X5R; SPN (none) -> 80-C0603C474K4P; SPR (none) -> Mouser
- C4, C5, C6, C7, C8: MFR (none) -> KEMET; MPN (none) -> C0603C104K3RECTU; Rating (none) -> 16V X5R; SPN (none) -> 80-C0603C104K3REC; SPR (none) -> Mouser
- D1: MFR (none) -> OnSemi; MPN (none) -> BAT54CLT3G; SPN (none) -> 863-BAT54CLT3G; SPR (none) -> Mouser
- D2: value LED -> LED_R; MFR (none) -> Wurth Electronics; MPN (none) -> 150060SS75000; SPN (none) -> 710-150060SS75000; SPR (none) -> Mouser
- D3, D4: value LED -> LED_Y; MFR (none) -> Wurth Electronics; MPN (none) -> 150060YS75000; SPN (none) -> 710-150060YS75000; SPR (none) -> Mouser
- F1, F2: MFR (none) -> Bel Fuse; MPN (none) -> C2Q 1.5; Rating (none) -> 1.5A; SPN (none) -> 530-C2Q1.5; SPR (none) -> Mouser
- J1: MFR (none) -> Molex; MPN (none) -> 504050-0591; SPN (none) -> 538-504050-0591; SPR (none) -> Mouser
- R1, R4, R5: MFR (none) -> Yageo; MPN (none) -> RC0603JR-133K3L; Rating (none) -> 1/10W 5%; SPN (none) -> 603-RC0603JR-133K3L; SPR (none) -> Mouser
- R10: MFR (none) -> Yageo; MPN (none) -> RC0603JR-070RL; Rating (none) -> 1/10W 5%; SPN (none) -> 603-RC0603JR-070RL; SPR (none) -> Mouser
- R2, R3, R7, R8: MFR (none) -> Yageo; MPN (none) -> RC0603FR-0710KL; Rating (none) -> 1/10W 5%; SPN (none) -> 603-RC0603FR-0710KL; SPR (none) -> Mouser
- R6: MFR (none) -> Yageo; MPN (none) -> RC0603FR-10470RL; Rating (none) -> 1/10W 5%; SPN (none) -> 603-RC0603FR-10470RL; SPR (none) -> Mouser
- U1: MFR (none) -> Microchip; MPN (none) -> MCP1703T-3302E/MB; SPN (none) -> 579-MCP1703T-3302EMB; SPR (none) -> Mouser
- U2: MFR (none) -> Microchip; MPN (none) -> PIC18LF45K50-I/PT; SPN (none) -> 579-PIC18LF45K50I/PT; SPR (none) -> Mouser
- U3: MFR (none) -> ISSI; MPN (none) -> IS61LV256AL-10TLI; SPN (none) -> 870-IS61LV256AL10TLI; SPR (none) -> Mouser
