File: GB-LIVE32/usb.sch (KiCad schematic (older format))
At the start: 6 parts, among them J2 USB_B_Mini

Commit message: BOM + docs
Parts:
- C10, C9: MFR (none) -> KEMET; MPN (none) -> C0603C104K3RECTU; Rating (none) -> 16V X5R; SPN (none) -> 80-C0603C104K3REC; SPR (none) -> Mouser
- C11: MFR (none) -> Taiyo Yuden; MPN (none) -> EMK212BJ475MD-T; Rating (none) -> 16V X5R; SPN (none) -> 963-EMK212BJ475MD-T; SPR (none) -> Mouser
- J2: MFR (none) -> Hirose; MPN (none) -> UX60SC-MB-5ST(80); SPN (none) -> 798-UX60SC-MB-5ST80; SPR (none) -> Mouser
- L1: MFR (none) -> TDK; MPN (none) -> MMZ1608Y601BTD25; SPN (none) -> 810-MMZ1608Y601BTD25; SPR (none) -> Mouser
Changed lines of the file:
@@
 F 2 "Capacitor_SMD:C_0603_1608Metric" H 6638 3700 50  0001 C CNN
 F 3 "~" H 6600 3850 50  0001 C CNN
+F 4 "Mouser" H 0   0   50  0001 C CNN "SPR"
+F 5 "KEMET" H 0   0   50  0001 C CNN "MFR"
+F 6 "C0603C104K3RECTU" H 0   0   50  0001 C CNN "MPN"
+F 7 "16V X5R" H 0   0   50  0001 C CNN "Rating"
+F 8 "80-C0603C104K3REC" H 0   0   50  0001 C CNN "SPN"
 	1    6600 3850
 	1    0    0    -1
@@
 F 2 "Capacitor_SMD:C_0603_1608Metric" H 5888 3700 50  0001 C CNN
 F 3 "~" H 5850 3850 50  0001 C CNN
+F 4 "Mouser" H 0   0   50  0001 C CNN "SPR"
+F 5 "KEMET" H 0   0   50  0001 C CNN "MFR"
+F 6 "C0603C104K3RECTU" H 0   0   50  0001 C CNN "MPN"
+F 7 "16V X5R" H 0   0   50  0001 C CNN "Rating"
+F 8 "80-C0603C104K3REC" H 0   0   50  0001 C CNN "SPN"
 	1    5850 3850
 	1    0    0    -1
@@
 F 2 "Inductor_SMD:L_0603_1608Metric" V 6180 3700 50  0001 C CNN
 F 3 "~" H 6250 3700 50  0001 C CNN
+F 4 "TDK" H 0   0   50  0001 C CNN "MFR"
+F 5 "MMZ1608Y601BTD25" H 0   0   50  0001 C CNN "MPN"
+F 6 "810-MMZ1608Y601BTD25" H 0   0   50  0001 C CNN "SPN"
+F 7 "Mouser" H 0   0   50  0001 C CNN "SPR"
 	1    6250 3700
 	0    1    1    0
@@
 F 2 "Gekkio_Connector_USB:USB_Mini-B_Hirose_UX60SC-MB-5ST80_Horizontal" H 5050 3850 50  0001 C CNN
 F 3 "~" H 5050 3850 50  0001 C CNN
+F 4 "Hirose" H 0   0   50  0001 C CNN "MFR"
+F 5 "UX60SC-MB-5ST(80)" H 0   0   50  0001 C CNN "MPN"
+F 6 "798-UX60SC-MB-5ST80" H 0   0   50  0001 C CNN "SPN"
+F 7 "Mouser" H 0   0   50  0001 C CNN "SPR"
 	1    4900 3900
 	1    0    0    -1
@@
 F 2 "Capacitor_SMD:C_0805_2012Metric" H 7088 3700 50  0001 C CNN
 F 3 "~" H 7050 3850 50  0001 C CNN
+F 4 "Mouser" H 0   0   50  0001 C CNN "SPR"
+F 5 "Taiyo Yuden" H 0   0   50  0001 C CNN "MFR"
+F 6 "EMK212BJ475MD-T" H 0   0   50  0001 C CNN "MPN"
+F 7 "16V X5R" H 0   0   50  0001 C CNN "Rating"
+F 8 "963-EMK212BJ475MD-T" H 0   0   50  0001 C CNN "SPN"
 	1    7050 3850
 	-1   0    0    1
