File: GB-LIVE32/gameboy.sch (KiCad schematic (older format))
At the start: 16 parts, among them J3 GameBoy_Cartridge, U4 74LVC1G32, U5 74LVC8T245PW, U6 74LVCH245APW, U7 74LVCH245APW, U8 74LVC1G32, U9 74LVC1G07

Commit message: BOM + docs
Parts:
- C12, C13, C14, C15, C16, C17, C18: MFR (none) -> KEMET; MPN (none) -> C0603C104K3RECTU; Rating (none) -> 16V X5R; SPN (none) -> 80-C0603C104K3REC; SPR (none) -> Mouser
- R9: MFR (none) -> Yageo; MPN (none) -> RC0603FR-0710KL; Rating (none) -> 1/10W 5%; SPN (none) -> 603-RC0603FR-0710KL; SPR (none) -> Mouser
- U4, U8: MFR (none) -> Nexperia; MPN (none) -> 74LVC1G32GW,125; SPN (none) -> 771-74LVC1G32GW-G; SPR (none) -> Mouser
- U5: MFR (none) -> Nexperia; MPN (none) -> 74LVCH8T245PW,118; SPN (none) -> 771-74LVCH8T245PW118; SPR (none) -> Mouser
- U6, U7: MFR (none) -> Nexperia; MPN (none) -> 74LVCH245APW,118; SPN (none) -> 771-74LVCH245APW-T; SPR (none) -> Mouser
- U9: MFR (none) -> Nexperia; MPN (none) -> 74LVC1G07GW,125; SPN (none) -> 771-74LVC1G07GW-G; SPR (none) -> Mouser
Changed lines of the file:
@@
 F 2 "Package_SO:TSSOP-20_4.4x6.5mm_P0.65mm" H 5700 1500 50  0001 C CNN
 F 3 "https://assets.nexperia.com/documents/data-sheet/74LVC_LVCH245A.pdf" H 5800 3050 50  0001 C CNN
+F 4 "Nexperia" H 0   0   50  0001 C CNN "MFR"
+F 5 "74LVCH245APW,118" H 0   0   50  0001 C CNN "MPN"
+F 6 "771-74LVCH245APW-T" H 0   0   50  0001 C CNN "SPN"
+F 7 "Mouser" H 0   0   50  0001 C CNN "SPR"
 	1    5700 2700
 	1    0    0    -1
@@
 F 2 "Package_SO:TSSOP-20_4.4x6.5mm_P0.65mm" H 8200 1500 50  0001 C CNN
 F 3 "https://assets.nexperia.com/documents/data-sheet/74LVC_LVCH245A.pdf" H 8300 3050 50  0001 C CNN
+F 4 "Nexperia" H 0   0   50  0001 C CNN "MFR"
+F 5 "74LVCH245APW,118" H 0   0   50  0001 C CNN "MPN"
+F 6 "771-74LVCH245APW-T" H 0   0   50  0001 C CNN "SPN"
+F 7 "Mouser" H 0   0   50  0001 C CNN "SPR"
 	1    8200 2700
 	1    0    0    -1
@@
 F 2 "Capacitor_SMD:C_0603_1608Metric" H 10038 5800 50  0001 C CNN
 F 3 "~" H 10000 5950 50  0001 C CNN
+F 4 "Mouser" H 0   0   50  0001 C CNN "SPR"
+F 5 "KEMET" H 0   0   50  0001 C CNN "MFR"
+F 6 "C0603C104K3RECTU" H 0   0   50  0001 C CNN "MPN"
+F 7 "16V X5R" H 0   0   50  0001 C CNN "Rating"
+F 8 "80-C0603C104K3REC" H 0   0   50  0001 C CNN "SPN"
 	1    10000 5950
 	1    0    0    -1
@@
 F 2 "Capacitor_SMD:C_0603_1608Metric" H 10538 5800 50  0001 C CNN
 F 3 "~" H 10500 5950 50  0001 C CNN
+F 4 "Mouser" H 0   0   50  0001 C CNN "SPR"
+F 5 "KEMET" H 0   0   50  0001 C CNN "MFR"
+F 6 "C0603C104K3RECTU" H 0   0   50  0001 C CNN "MPN"
+F 7 "16V X5R" H 0   0   50  0001 C CNN "Rating"
+F 8 "80-C0603C104K3REC" H 0   0   50  0001 C CNN "SPN"
 	1    10500 5950
 	1    0    0    -1
@@
 F 2 "Capacitor_SMD:C_0603_1608Metric" H 9538 5800 50  0001 C CNN
 F 3 "~" H 9500 5950 50  0001 C CNN
+F 4 "Mouser" H 0   0   50  0001 C CNN "SPR"
+F 5 "KEMET" H 0   0   50  0001 C CNN "MFR"
+F 6 "C0603C104K3RECTU" H 0   0   50  0001 C CNN "MPN"
+F 7 "16V X5R" H 0   0   50  0001 C CNN "Rating"
+F 8 "80-C0603C104K3REC" H 0   0   50  0001 C CNN "SPN"
 	1    9500 5950
 	1    0    0    -1
@@
 F 2 "Capacitor_SMD:C_0603_1608Metric" H 9038 5800 50  0001 C CNN
 F 3 "~" H 9000 5950 50  0001 C CNN
+F 4 "Mouser" H 0   0   50  0001 C CNN "SPR"
+F 5 "KEMET" H 0   0   50  0001 C CNN "MFR"
+F 6 "C0603C104K3RECTU" H 0   0   50  0001 C CNN "MPN"
+F 7 "16V X5R" H 0   0   50  0001 C CNN "Rating"
+F 8 "80-C0603C104K3REC" H 0   0   50  0001 C CNN "SPN"
 	1    9000 5950
 	1    0    0    -1
@@
 F 2 "Package_TO_SOT_SMD:SOT-353_SC-70-5" H 8400 1450 50  0001 C CNN
 F 3 "http://www.ti.com/lit/sg/scyt129e/scyt129e.pdf" H 8400 1450 50  0001 C CNN
+F 4 "Mouser" H 0   0   50  0001 C CNN "SPR"
+F 5 "Nexperia" H 0   0   50  0001 C CNN "MFR"
+F 6 "74LVC1G32GW,125" H 0   0   50  0001 C CNN "MPN"
+F 7 "771-74LVC1G32GW-G" H 0   0   50  0001 C CNN "SPN"
 	1    8400 1450
 	-1   0    0    -1
@@
 F 2 "Capacitor_SMD:C_0603_1608Metric" H 8538 5800 50  0001 C CNN
 F 3 "~" H 8500 5950 50  0001 C CNN
+F 4 "Mouser" H 0   0   50  0001 C CNN "SPR"
+F 5 "KEMET" H 0   0   50  0001 C CNN "MFR"
+F 6 "C0603C104K3RECTU" H 0   0   50  0001 C CNN "MPN"
+F 7 "16V X5R" H 0   0   50  0001 C CNN "Rating"
+F 8 "80-C0603C104K3REC" H 0   0   50  0001 C CNN "SPN"
 	1    8500 5950
 	1    0    0    -1
@@
 F 2 "Package_TO_SOT_SMD:SOT-353_SC-70-5" H 8750 4500 50  0001 C CNN
 F 3 "http://www.ti.com/lit/sg/scyt129e/scyt129e.pdf" H 8750 4500 50  0001 C CNN
+F 4 "Mouser" H 0   0   50  0001 C CNN "SPR"
+F 5 "Nexperia" H 0   0   50  0001 C CNN "MFR"
+F 6 "74LVC1G07GW,125" H 0   0   50  0001 C CNN "MPN"
+F 7 "771-74LVC1G07GW-G" H 0   0   50  0001 C CNN "SPN"
 	1    8750 4500
 	1    0    0    -1
@@
 F 2 "Capacitor_SMD:C_0603_1608Metric" H 8038 5800 50  0001 C CNN
 F 3 "~" H 8000 5950 50  0001 C CNN
+F 4 "Mouser" H 0   0   50  0001 C CNN "SPR"
+F 5 "KEMET" H 0   0   50  0001 C CNN "MFR"
+F 6 "C0603C104K3RECTU" H 0   0   50  0001 C CNN "MPN"
+F 7 "16V X5R" H 0   0   50  0001 C CNN "Rating"
+F 8 "80-C0603C104K3REC" H 0   0   50  0001 C CNN "SPN"
 	1    8000 5950
 	1    0    0    -1
@@
 F 2 "Capacitor_SMD:C_0603_1608Metric" H 7538 5800 50  0001 C CNN
 F 3 "~" H 7500 5950 50  0001 C CNN
+F 4 "Mouser" H 0   0   50  0001 C CNN "SPR"
+F 5 "KEMET" H 0   0   50  0001 C CNN "MFR"
+F 6 "C0603C104K3RECTU" H 0   0   50  0001 C CNN "MPN"
+F 7 "16V X5R" H 0   0   50  0001 C CNN "Rating"
+F 8 "80-C0603C104K3REC" H 0   0   50  0001 C CNN "SPN"
 	1    7500 5950
 	1    0    0    -1
@@
 F 2 "Package_SO:TSSOP-24_4.4x7.8mm_P0.65mm" H 3100 1500 50  0001 C CNN
 F 3 "https://assets.nexperia.com/documents/data-sheet/74LVC_LVCH8T245.pdf" H 3200 3050 50  0001 C CNN
+F 4 "Nexperia" H 0   0   50  0001 C CNN "MFR"
+F 5 "74LVCH8T245PW,118" H 0   0   50  0001 C CNN "MPN"
+F 6 "771-74LVCH8T245PW118" H 0   0   50  0001 C CNN "SPN"
+F 7 "Mouser" H 0   0   50  0001 C CNN "SPR"
 	1    3100 2700
 	1    0    0    -1
@@
 F 2 "Package_TO_SOT_SMD:SOT-353_SC-70-5" H 1550 3200 50  0001 C CNN
 F 3 "http://www.ti.com/lit/sg/scyt129e/scyt129e.pdf" H 1550 3200 50  0001 C CNN
+F 4 "Mouser" H 0   0   50  0001 C CNN "SPR"
+F 5 "Nexperia" H 0   0   50  0001 C CNN "MFR"
+F 6 "74LVC1G32GW,125" H 0   0   50  0001 C CNN "MPN"
+F 7 "771-74LVC1G32GW-G" H 0   0   50  0001 C CNN "SPN"
 	1    1550 3200
 	1    0    0    -1
@@
 F 2 "Resistor_SMD:R_0603_1608Metric" V 8130 4350 50  0001 C CNN
 F 3 "~" H 8200 4350 50  0001 C CNN
+F 4 "Yageo" H 0   0   50  0001 C CNN "MFR"
+F 5 "RC0603FR-0710KL" H 0   0   50  0001 C CNN "MPN"
+F 6 "603-RC0603FR-0710KL" H 0   0   50  0001 C CNN "SPN"
+F 7 "Mouser" H 0   0   50  0001 C CNN "SPR"
+F 8 "1/10W 5%" H 0   0   50  0001 C CNN "Rating"
 	1    8200 4350
 	1    0    0    -1

Commit message: More BOM stuff
Parts:
- J3: value GameBoy_Cartridge -> DNF
Changed lines of the file:
@@
 P 10200 2800
 F 0 "J3" H 10430 2850 50  0000 L CNN
-F 1 "GameBoy_Cartridge" H 10430 2759 50  0000 L CNN
+F 1 "DNF" H 10430 2759 50  0000 L CNN
 F 2 "Gekkio_Connector_PCBEdge:GameBoy_Cartridge_1x32_P1.50mm_Edge" H 10100 1000 50  0001 C CNN
 F 3 "" H 10100 2800 50  0001 L CNN

Commit message: Stop recommending bus hold transceivers for GB-LIVE32 boards
Parts:
- U5: MPN 74LVCH8T245PW,118 -> 74LVC8T245PW,118; SPN 771-74LVCH8T245PW118 -> 771-74LVC8T245PW118
- U6, U7: value 74LVCH245APW -> 74LVC245APW; symbol Gekkio_Logic_LevelTranslator:74LVCH245APW -> Gekkio_Logic_LevelTranslator:74LVC245APW; MPN 74LVCH245APW,118 -> 74LVC245APW,118; SPN 771-74LVCH245APW-T -> 771-74LVC245APW-T
Changed lines of the file:
@@
 $EndComp
 $Comp
-L Gekkio_Logic_LevelTranslator:74LVCH245APW U6
+L Gekkio_Logic_LevelTranslator:74LVC245APW U6
 U 1 1 5AEA9A8F
 P 5700 2700
 F 0 "U6" H 5500 3500 50  0000 C CNN
-F 1 "74LVCH245APW" H 5250 3400 50  0000 C CNN
+F 1 "74LVC245APW" H 5250 3400 50  0000 C CNN
 F 2 "Package_SO:TSSOP-20_4.4x6.5mm_P0.65mm" H 5700 1500 50  0001 C CNN
-F 3 "https://assets.nexperia.com/documents/data-sheet/74LVC_LVCH245A.pdf" H 5800 3050 50  0001 C CNN
+F 3 "" H 5800 3050 50  0001 C CNN
 F 4 "Nexperia" H 0   0   50  0001 C CNN "MFR"
-F 5 "74LVCH245APW,118" H 0   0   50  0001 C CNN "MPN"
-F 6 "771-74LVCH245APW-T" H 0   0   50  0001 C CNN "SPN"
+F 5 "74LVC245APW,118" H 0   0   50  0001 C CNN "MPN"
+F 6 "771-74LVC245APW-T" H 0   0   50  0001 C CNN "SPN"
 F 7 "Mouser" H 0   0   50  0001 C CNN "SPR"
 	1    5700 2700
@@
 	6700 2800 6800 2900
 $Comp
-L Gekkio_Logic_LevelTranslator:74LVCH245APW U7
+L Gekkio_Logic_LevelTranslator:74LVC245APW U7
 U 1 1 5AECA2B3
 P 8200 2700
 F 0 "U7" H 8000 3500 50  0000 C CNN
-F 1 "74LVCH245APW" H 7750 3400 50  0000 C CNN
+F 1 "74LVC245APW" H 7750 3400 50  0000 C CNN
 F 2 "Package_SO:TSSOP-20_4.4x6.5mm_P0.65mm" H 8200 1500 50  0001 C CNN
-F 3 "https://assets.nexperia.com/documents/data-sheet/74LVC_LVCH245A.pdf" H 8300 3050 50  0001 C CNN
+F 3 "" H 8300 3050 50  0001 C CNN
 F 4 "Nexperia" H 0   0   50  0001 C CNN "MFR"
-F 5 "74LVCH245APW,118" H 0   0   50  0001 C CNN "MPN"
-F 6 "771-74LVCH245APW-T" H 0   0   50  0001 C CNN "SPN"
+F 5 "74LVC245APW,118" H 0   0   50  0001 C CNN "MPN"
+F 6 "771-74LVC245APW-T" H 0   0   50  0001 C CNN "SPN"
 F 7 "Mouser" H 0   0   50  0001 C CNN "SPR"
 	1    8200 2700
@@
 F 1 "74LVC8T245PW" H 2500 3400 50  0000 C CNN
 F 2 "Package_SO:TSSOP-24_4.4x7.8mm_P0.65mm" H 3100 1500 50  0001 C CNN
-F 3 "https://assets.nexperia.com/documents/data-sheet/74LVC_LVCH8T245.pdf" H 3200 3050 50  0001 C CNN
+F 3 "" H 3200 3050 50  0001 C CNN
 F 4 "Nexperia" H 0   0   50  0001 C CNN "MFR"
-F 5 "74LVCH8T245PW,118" H 0   0   50  0001 C CNN "MPN"
-F 6 "771-74LVCH8T245PW118" H 0   0   50  0001 C CNN "SPN"
+F 5 "74LVC8T245PW,118" H 0   0   50  0001 C CNN "MPN"
+F 6 "771-74LVC8T245PW118" H 0   0   50  0001 C CNN "SPN"
 F 7 "Mouser" H 0   0   50  0001 C CNN "SPR"
 	1    3100 2700
