File: GB-LIVE32/GB-LIVE32.kicad_pcb (KiCad board)
At the start: 4 copper layers, 51.4 x 61 mm, 61 parts, among them J1 Conn_01x05, J2 USB_B_Mini, J3 GameBoy_Cartridge, U1 MCP1703A-3302_SOT89, U2 PIC18LF45K50_QFP, U3 IS61LV256AL-10T, U4 74LVC1G32, U5 74LVC8T245PW, U6 74LVCH245APW, U7 74LVCH245APW, U8 74LVC1G32, U9 74LVC1G07

Commit message: More details and fixes
Other:
- board text added: "PCB size: 51.4x61mm PCB thickness: 0.8mm"
Changed lines of the file:
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@@
-(kicad_pcb (version 20171130) (host pcbnew 5.0.0-rc2-unknown-01c2d93~65~ubuntu18.04.1)
+(kicad_pcb (version 20171130) (host pcbnew 5.0.0-rc3-unknown-101b68b~65~ubuntu18.04.1)
   (general
-    (thickness 1.6)
-    (drawings 11)
+    (thickness 0.8)
+    (drawings 17)
     (tracks 935)
     (zones 0)
@@
   (layers
     (0 F.Cu signal)
-    (1 In1.Cu signal hide)
-    (2 In2.Cu signal hide)
+    (1 In1.Cu signal)
+    (2 In2.Cu signal)
     (31 B.Cu signal)
     (32 B.Adhes user)
@@
     )
   )
+  (gr_text "PCB size: 51.4x61mm\nPCB thickness: 0.8mm" (at 127 104) (layer F.Fab)
+    (effects (font (size 1.5 1.5) (thickness 0.3)) (justify left))
+  )
+  (dimension 51.4 (width 0.3) (layer F.Fab)
+    (gr_text "51,400 mm" (at 100 32.8) (layer F.Fab)
+      (effects (font (size 1.5 1.5) (thickness 0.3)))
+    )
+    (feature1 (pts (xy 125.7 38) (xy 125.7 34.313579)))
+    (feature2 (pts (xy 74.3 38) (xy 74.3 34.313579)))
+    (crossbar (pts (xy 74.3 34.9) (xy 125.7 34.9)))
+    (arrow1a (pts (xy 125.7 34.9) (xy 124.573496 35.486421)))
+    (arrow1b (pts (xy 125.7 34.9) (xy 124.573496 34.313579)))
+    (arrow2a (pts (xy 74.3 34.9) (xy 75.426504 35.486421)))
+    (arrow2b (pts (xy 74.3 34.9) (xy 75.426504 34.313579)))
+  )
+  (dimension 8.6 (width 0.2) (layer F.Fab)
+    (gr_text "8,600 mm" (at 71.4 95.7 270) (layer F.Fab)
+      (effects (font (size 1 1) (thickness 0.2)))
+    )
+    (feature1 (pts (xy 73.9 100) (xy 72.213579 100)))
+    (feature2 (pts (xy 73.9 91.4) (xy 72.213579 91.4)))
+    (crossbar (pts (xy 72.8 91.4) (xy 72.8 100)))
+    (arrow1a (pts (xy 72.8 100) (xy 72.213579 98.873496)))
+    (arrow1b (pts (xy 72.8 100) (xy 73.386421 98.873496)))
+    (arrow2a (pts (xy 72.8 91.4) (xy 72.213579 92.526504)))
+    (arrow2b (pts (xy 72.8 91.4) (xy 73.386421 92.526504)))
+  )
+  (dimension 52.4 (width 0.3) (layer F.Fab)
+    (gr_text "52,400 mm" (at 66.5 65.2 270) (layer F.Fab)
+      (effects (font (size 1.5 1.5) (thickness 0.3)))
+    )
+    (feature1 (pts (xy 70.6 91.4) (xy 68.013579 91.4)))
+    (feature2 (pts (xy 70.6 39) (xy 68.013579 39)))
+    (crossbar (pts (xy 68.6 39) (xy 68.6 91.4)))
+    (arrow1a (pts (xy 68.6 91.4) (xy 68.013579 90.273496)))
+    (arrow1b (pts (xy 68.6 91.4) (xy 69.186421 90.273496)))
+    (arrow2a (pts (xy 68.6 39) (xy 68.013579 40.126504)))
+    (arrow2b (pts (xy 68.6 39) (xy 69.186421 40.126504)))
+  )
+  (dimension 61 (width 0.3) (layer F.Fab)
+    (gr_text "61,000 mm" (at 134.7 69.5 270) (layer F.Fab)
+      (effects (font (size 1.5 1.5) (thickness 0.3)))
+    )
+    (feature1 (pts (xy 127 100) (xy 133.186421 100)))
+    (feature2 (pts (xy 127 39) (xy 133.186421 39)))
+    (crossbar (pts (xy 132.6 39) (xy 132.6 100)))
+    (arrow1a (pts (xy 132.6 100) (xy 132.013579 98.873496)))
+    (arrow1b (pts (xy 132.6 100) (xy 133.186421 98.873496)))
+    (arrow2a (pts (xy 132.6 39) (xy 132.013579 40.126504)))
+    (arrow2b (pts (xy 132.6 39) (xy 133.186421 40.126504)))
+  )
+  (dimension 49.2 (width 0.3) (layer F.Fab)
+    (gr_text "49,200 mm" (at 100 106.9) (layer F.Fab)
+      (effects (font (size 1.5 1.5) (thickness 0.3)))
+    )
+    (feature1 (pts (xy 124.6 100.5) (xy 124.6 105.386421)))
+    (feature2 (pts (xy 75.4 100.5) (xy 75.4 105.386421)))
+    (crossbar (pts (xy 75.4 104.8) (xy 124.6 104.8)))
+    (arrow1a (pts (xy 124.6 104.8) (xy 123.473496 105.386421)))
+    (arrow1b (pts (xy 124.6 104.8) (xy 123.473496 104.213579)))
+    (arrow2a (pts (xy 75.4 104.8) (xy 76.526504 105.386421)))
+    (arrow2b (pts (xy 75.4 104.8) (xy 76.526504 104.213579)))
+  )
   (gr_text "GB-LIVE32 v2.0\nhttps://gekkio.fi" (at 116.7 75.9) (layer F.SilkS)

Commit message: BOM + docs
Parts:
- D2: value LED -> LED_R
- D3, D4: value LED -> LED_Y
Changed lines of the file:
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@@
       (effects (font (size 1 1) (thickness 0.15)))
     )
-    (fp_text value LED (at 0 1.45 90) (layer F.Fab) hide
+    (fp_text value LED_R (at 0 1.45 90) (layer F.Fab) hide
       (effects (font (size 1 1) (thickness 0.15)))
     )
@@
       (effects (font (size 1 1) (thickness 0.15)))
     )
-    (fp_text value LED (at 0 1.45 270) (layer F.Fab) hide
+    (fp_text value LED_Y (at 0 1.45 270) (layer F.Fab) hide
       (effects (font (size 1 1) (thickness 0.15)))
     )
@@
       (effects (font (size 1 1) (thickness 0.15)))
     )
-    (fp_text value LED (at 0 1.45 270) (layer F.Fab) hide
+    (fp_text value LED_Y (at 0 1.45 270) (layer F.Fab) hide
       (effects (font (size 1 1) (thickness 0.15)))
     )

Commit message: More BOM stuff
Parts:
- J3: value GameBoy_Cartridge -> DNF
Changed lines of the file:
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@@
       (effects (font (size 1 1) (thickness 0.15)))
     )
-    (fp_text value GameBoy_Cartridge (at 0 -8) (layer F.Fab) hide
+    (fp_text value DNF (at 0 -8) (layer F.Fab) hide
       (effects (font (size 1 1) (thickness 0.15)))
     )

Commit message: Stop recommending bus hold transceivers for GB-LIVE32 boards
Parts:
- U6, U7: value 74LVCH245APW -> 74LVC245APW
Changed lines of the file:
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@@
-(kicad_pcb (version 20171130) (host pcbnew 5.0.0-rc3-unknown-101b68b~65~ubuntu18.04.1)
+(kicad_pcb (version 20171130) (host pcbnew 5.0.0-rc3-unknown-14ce5182~65~ubuntu18.04.1)
   (general
     (thickness 0.8)
@@
       (effects (font (size 1 1) (thickness 0.15)))
     )
-    (fp_text value 74LVCH245APW (at 0 4.3 270) (layer F.Fab) hide
+    (fp_text value 74LVC245APW (at 0 4.3 270) (layer F.Fab) hide
       (effects (font (size 1 1) (thickness 0.15)))
     )
@@
       (effects (font (size 1 1) (thickness 0.15)))
     )
-    (fp_text value 74LVCH245APW (at 0 4.3 270) (layer F.Fab) hide
-      (effects (font (size 1 1) (thickness 0.15)))
-    )
+    (fp_text value 74LVC245APW (at 0 4.3 270) (layer F.Fab) hide
+      (effects (font (size 1 1) (thickness 0.15)))
+    )

Commit message: Update PCB size and thickness recommendations
Other:
- board text added: "PCB size: 51.4x61mm PCB thickness: 1.0mm"
- board text removed: "PCB size: 51.4x61mm PCB thickness: 0.8mm"
Changed lines of the file:
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@@
-(kicad_pcb (version 20171130) (host pcbnew 5.0.0-rc3-unknown-14ce5182~65~ubuntu18.04.1)
+(kicad_pcb (version 20171130) (host pcbnew 5.0.2-bee76a0~70~ubuntu18.10.1)
   (general
-    (thickness 0.8)
+    (thickness 1)
     (drawings 17)
     (tracks 935)
@@
     )
   )
-  (gr_text "PCB size: 51.4x61mm\nPCB thickness: 0.8mm" (at 127 104) (layer F.Fab)
+  (gr_text "PCB size: 51.4x61mm\nPCB thickness: 1.0mm" (at 127 104) (layer F.Fab)
     (effects (font (size 1.5 1.5) (thickness 0.3)) (justify left))
   )

Commit message: Adjust solder mask clearances, regenerate gerbers
Other:
- rule pad_to_mask_clearance: 0.2 -> 0
Changed lines of the file:
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@@
     (pad_size 2 2)
     (pad_drill 0)
-    (pad_to_mask_clearance 0.2)
+    (pad_to_mask_clearance 0)
     (solder_mask_min_width 0.2)
     (aux_axis_origin 0 0)
@@
       (usegerberattributes false)
       (usegerberadvancedattributes false)
-      (creategerberjobfile false)
+      (creategerberjobfile true)
       (excludeedgelayer false)
       (linewidth 0.100000)

Commit message: Upgrade most projects to KiCad 6
Parts:
- TP10: value ~OE -> ~{OE}
- TP12: value ~RES -> ~{RES}
- TP7: value ~CS -> ~{CS}
- TP8: value ~GB_EN -> ~{GB_EN}
- TP9: value ~WR -> ~{WR}
Connections:
- net /gameboy/~GB_RD renamed /gameboy/~{GB_RD}
- net /gameboy/~GB_RES renamed /gameboy/~{GB_RES}
- net /~CS renamed /~{CS}
- net /~GB_EN renamed /~{GB_EN}
- net /~GB_RES renamed /~{GB_RES}
- net /~OE renamed /~{OE}
- net /~WR renamed /~{WR}
Other:
- net class Default removed
- net class Power removed
