File: GB-CART2M-A/GB-CART2M-A.kicad_pcb (KiCad board)
At the start: 2 copper layers, 51.4 x 61 mm, 28 parts, among them J1 Conn_02x05_Odd_Even, J2 GameBoy_Cartridge, U1 LC4032ZE-XXTN48, U2 MIC5370, U3 AT49F002-xxJx

Commit message: Update PCB size and thickness recommendations
Other:
- board text added: "PCB size: 51.4x61mm PCB thickness: 1.0mm"
- board text removed: "PCB size: 51.4x61mm PCB thickness: 0.8mm"
Changed lines of the file:
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@@
 (kicad_pcb (version 20171130) (host pcbnew 5.0.2-bee76a0~70~ubuntu18.10.1)
   (general
-    (thickness 0.8)
+    (thickness 1)
     (drawings 23)
     (tracks 731)
@@
     (effects (font (size 1.2 1.2) (thickness 0.2)))
   )
-  (gr_text "PCB size: 51.4x61mm\nPCB thickness: 0.8mm" (at 127 104) (layer F.Fab)
+  (gr_text "PCB size: 51.4x61mm\nPCB thickness: 1.0mm" (at 127 104) (layer F.Fab)
     (effects (font (size 1.5 1.5) (thickness 0.3)) (justify left))
   )

Commit message: Add GB-CART2M-A v1.1
Parts:
- removed the TP2 at (106.5, 46.0)
- removed TP4: TestPoint, TestPoint:TestPoint_THTPad_D2.0mm_Drill1.0mm
- C10, C4, C6, C7, C9: value 0.1uF -> 100nF
- J1: value Conn_02x05_Odd_Even -> Conn_02x05_Counter_Clockwise; footprint Connector_PinHeader_1.27mm:PinHeader_2x05_P1.27mm_Vertical -> Connector:Tag-Connect_TC2050-IDC-NL_2x05_P1.27mm_Vertical
- J2: value GameBoy_Cartridge -> DNF
- JP1, JP2: value Jumper_NC_Small -> DNF
- R4: value R -> 47k
- moved R3 5.82 mm to (104.9, 44.5)
- moved R1 3.73 mm to (116.1, 44.5)
- moved J1 2.34 mm to (110.5, 44.0), turned to 0 degrees
- renumbered TP3 to TP2, TP5 to TP3
Connections:
- J1 pad 2: GND -> /TDO
- J1 pad 3: /TDO -> /TMS
- J1 pad 4: +1V8 -> (no net)
- J1 pad 5: /TMS -> /TDI
- J1 pad 6: Net-(J1-Pad6) -> GND
- J1 pad 7: Net-(J1-Pad7) -> (no net)
- J1 pad 8: Net-(J1-Pad8) -> (no net)
- J1 pad 9: /TDI -> +1V8
- J2 pad 2: Net-(J2-Pad2) -> (no net)
- J2 pad 5: Net-(J2-Pad5) -> (no net)
- U1 pad 28: Net-(U1-Pad28) -> (no net)
- U1 pad 31: Net-(U1-Pad31) -> (no net)
- U1 pad 32: Net-(U1-Pad32) -> (no net)
- U1 pad 38: Net-(U1-Pad38) -> (no net)
- U1 pad 39: Net-(U1-Pad39) -> (no net)
- U1 pad 4: Net-(U1-Pad4) -> (no net)
- U1 pad 40: Net-(U1-Pad40) -> (no net)
- U1 pad 41: Net-(U1-Pad41) -> (no net)
- U1 pad 44: Net-(TP2-Pad1) -> (no net)
- U1 pad 45: Net-(U1-Pad45) -> (no net)
- U1 pad 46: Net-(TP4-Pad1) -> (no net)
- U1 pad 47: Net-(U1-Pad47) -> (no net)
- U1 pad 48: Net-(U1-Pad48) -> (no net)
- U1 pad 7: Net-(U1-Pad7) -> (no net)
Routing:
- net Net-(TP4-Pad1): track 10.2 -> 0.00 mm, vias 2 -> 0
- net Net-(TP2-Pad1): track 8.42 -> 0.00 mm, vias 1 -> 0
- net +1V8: track 94.0 -> 99.2 mm
- net /TMS: track 14.2 -> 18.2 mm
- net /TDI: track 16.8 -> 13.7 mm, vias 3 -> 2
- net /TDO: track 11.6 -> 14.6 mm
- net GND: track 35.0 -> 37.0 mm, vias 16 -> 19
- net /TCK: track 17.4 -> 18.7 mm
Other:
- outline, holes or cut-outs redrawn
- board text added: "GB-CART2M-A v1.1 https://gekkio.fi"
- board text removed: "GB-CART2M-A v1.0 https://gekkio.fi"
