File: GB-BRK-CPU-G2/GB-BRK-CPU-G2.sch (KiCad schematic (older format))
At the start: 19 parts, among them J1 Conn_02x12_Top_Bottom, J2 Conn_02x08_Top_Bottom, J3 Conn_02x12_Top_Bottom, J4 Conn_02x08_Top_Bottom, J5 Conn_01x04, J6 Conn_01x04, U1 GameBoy_CPU_DMG-SGB

Commit message: Fix schematics broken after library updates
Parts:
- MK1, MK2, MK3, MK4: value Mounting_Hole_PAD -> MountingHole_Pad; symbol Mechanical:Mounting_Hole_PAD -> Mechanical:MountingHole_Pad
Changed lines of the file:
@@
 	4300 2200 4750 2200
 $Comp
-L Mechanical:Mounting_Hole_PAD MK1
+L Mechanical:MountingHole_Pad MK1
 U 1 1 5AFD33F1
 P 7100 1100
 F 0 "MK1" H 7200 1151 50  0000 L CNN
-F 1 "Mounting_Hole_PAD" H 7200 1060 50  0000 L CNN
+F 1 "MountingHole_Pad" H 7200 1060 50  0000 L CNN
 F 2 "MountingHole:MountingHole_3.2mm_M3_Pad_Via" H 7100 1100 50  0001 C CNN
 F 3 "" H 7100 1100 50  0001 C CNN
@@
 $EndComp
 $Comp
-L Mechanical:Mounting_Hole_PAD MK2
+L Mechanical:MountingHole_Pad MK2
 U 1 1 5AFD3497
 P 8100 1100
 F 0 "MK2" H 8200 1151 50  0000 L CNN
-F 1 "Mounting_Hole_PAD" H 8200 1060 50  0000 L CNN
+F 1 "MountingHole_Pad" H 8200 1060 50  0000 L CNN
 F 2 "MountingHole:MountingHole_3.2mm_M3_Pad_Via" H 8100 1100 50  0001 C CNN
 F 3 "" H 8100 1100 50  0001 C CNN
@@
 $EndComp
 $Comp
-L Mechanical:Mounting_Hole_PAD MK3
+L Mechanical:MountingHole_Pad MK3
 U 1 1 5AFD3565
 P 9100 1100
 F 0 "MK3" H 9200 1151 50  0000 L CNN
-F 1 "Mounting_Hole_PAD" H 9200 1060 50  0000 L CNN
+F 1 "MountingHole_Pad" H 9200 1060 50  0000 L CNN
 F 2 "MountingHole:MountingHole_3.2mm_M3_Pad_Via" H 9100 1100 50  0001 C CNN
 F 3 "" H 9100 1100 50  0001 C CNN
@@
 $EndComp
 $Comp
-L Mechanical:Mounting_Hole_PAD MK4
+L Mechanical:MountingHole_Pad MK4
 U 1 1 5AFD35D5
 P 10100 1100
 F 0 "MK4" H 10200 1151 50  0000 L CNN
-F 1 "Mounting_Hole_PAD" H 10200 1060 50  0000 L CNN
+F 1 "MountingHole_Pad" H 10200 1060 50  0000 L CNN
 F 2 "MountingHole:MountingHole_3.2mm_M3_Pad_Via" H 10100 1100 50  0001 C CNN
 F 3 "" H 10100 1100 50  0001 C CNN
@@
 	1    0    0    -1
 $EndComp
-Wire Wire Line
-	10100 1200 9100 1200
-Wire Wire Line
-	9100 1200 8100 1200
-Connection ~ 9100 1200
-Wire Wire Line
-	8100 1200 7100 1200
-Connection ~ 8100 1200
 $Comp
 L power:GND #PWR01
@@
 Wire Wire Line
 	7100 1200 7100 1300
-Connection ~ 7100 1200
 Wire Wire Line
 	2500 7200 2950 7200
@@
 Wire Wire Line
 	5400 1000 5900 1000
+Wire Wire Line
+	7100 1200 8100 1200
+Connection ~ 9100 1200
+Wire Wire Line
+	9100 1200 10100 1200
+Connection ~ 8100 1200
+Wire Wire Line
+	8100 1200 9100 1200
 $EndSCHEMATC

Commit message: Update GB-BRK-CPU-G1/G2
Connections:
- net Pin_27: now also U1.27 (SO1); no longer U1.28 (SO2)
- net Pin_28: now also U1.28 (SO2); no longer U1.27 (SO1)
Changed lines of the file:
@@
 EESchema Schematic File Version 4
 LIBS:GB-BRK-CPU-G2-cache
-EELAYER 26 0
+EELAYER 30 0
 EELAYER END
 $Descr A4 11693 8268
@@
 Title "GB-BRK-CPU-G2"
 Date ""
-Rev "v1.0"
+Rev "v1.1"
 Comp "https://gekkio.fi"
 Comment1 ""
@@
 Text Label 1800 5600 2    50   ~ 0
 Pin_26
+Text Label 1800 5800 2    50   ~ 0
+Pin_28
 Text Label 1800 5700 2    50   ~ 0
-Pin_28
-Text Label 1800 5800 2    50   ~ 0
 Pin_27
 Text Label 1800 6000 2    50   ~ 0
