File: GB-BENCH-G1/GB-BENCH-G1.kicad_pcb (KiCad board)
At the start: 4 copper layers, 100 x 100 mm, 98 parts, among them J1 BARREL_JACK, J10 CONN_01X06, J11 CONN_02X16, J12 CONN_01X06, J13 Conn_GameBoy_Cartridge_Slot, J14 CONN_01X05, J2 Conn_Molex_19708, J3 CONN_02X08, J4 CONN_02X08, J7 CONN_02X05, J8 CONN_02X13, J9 CONN_01X08, SW1 SW_SPST, U1 LC4256ZE-XXTN100, U2 MCP1703A-1802/MB, U3 MCP1703A-3302/MB, U4 MCP1703A-5002/MB, U5 LC4256ZE-XXTN100, U6 GameBoy_SRAM_64K, U7 GameBoy_SRAM_64K, U8 GameBoy_CPU_DMG-SGB, X1 XO32

Commit message: Adjust solder mask clearances, regenerate gerbers
Other:
- rule pad_to_mask_clearance: 0.2 -> 0

Commit message: Rescue GB-BENCH-G1 and convert to KiCad 6
Connections:
- net /~CS renamed /~{CS}
- net /~MCS renamed /~{MCS}
- net /~MRD renamed /~{MRD}
- net /~MWR renamed /~{MWR}
- net /~RD renamed /~{RD}
- net /~SYS_RD renamed /~{SYS_RD}
- net /~SYS_RST renamed /~{SYS_RST}
- net /~SYS_WR renamed /~{SYS_WR}
- net /~WR renamed /~{WR}
- net ~RES renamed ~{RES}
Other:
- net class Default removed
- net class Power removed
- board text added: "~{CS}"
- board text added: "~{MCS}"
- board text added: "~{MRD}"
- board text added: "~{MWR}"
- board text added: "~{RD}"
- board text added: "~{RES}"
- board text added: "~{WR}"
- board text removed: "~CS"
- board text removed: "~MCS"
- board text removed: "~MRD"
- board text removed: "~MWR"
- board text removed: "~RD"
- board text removed: "~RES"
- board text removed: "~WR"
