File: GB-BRK-CPU-G1/GB-BRK-CPU-G1.kicad_pcb (KiCad board)
At the start: 2 copper layers, 80 x 80 mm, 19 parts, among them J1 Conn_02x12_Top_Bottom, J2 Conn_02x08_Top_Bottom, J3 Conn_02x12_Top_Bottom, J4 Conn_02x08_Top_Bottom, J5 Conn_01x04, J6 Conn_01x04, U1 GameBoy_CPU_DMG-SGB

Commit message: Adjust solder mask clearances, regenerate gerbers
Other:
- rule pad_to_mask_clearance: 0.2 -> 0
Changed lines of the file:
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@@
-(kicad_pcb (version 20171130) (host pcbnew 5.0.0-fee4fd1~65~ubuntu18.04.1)
+(kicad_pcb (version 20171130) (host pcbnew 5.0.2-bee76a0~70~ubuntu18.10.1)
   (general
     (thickness 1.6)
@@
     (pad_size 1.524 1.524)
     (pad_drill 0.762)
-    (pad_to_mask_clearance 0.2)
+    (pad_to_mask_clearance 0)
     (solder_mask_min_width 0.2)
     (aux_axis_origin 0 0)
@@
       (usegerberattributes false)
       (usegerberadvancedattributes false)
-      (creategerberjobfile false)
+      (creategerberjobfile true)
       (excludeedgelayer false)
       (linewidth 0.100000)

Commit message: Update GB-BRK-CPU-G1/G2
Parts:
- MK1, MK2, MK3, MK4: value Mounting_Hole_PAD -> MountingHole_Pad
Other:
- outline, holes or cut-outs redrawn
- board text added: "CK1"
- board text added: "CK2"
- board text added: "GB-BRK-CPU-G1 v1.1 https://gekkio.fi"
- board text added: "S"
- board text added: "SCK"
- board text added: "SO1"
- board text added: "SO2"
- board text added: "ST"
- board text removed: "GB-BRK-CPU-G1 v1.0 https://gekkio.fi"
- board text removed: "HSYNC"
- board text removed: "LOUT"
- board text removed: "ROUT"
- board text removed: "SCLK"
- board text removed: "VSYNC"
- board text removed: "XI"
- board text removed: "XO"

Commit message: Upgrade most projects to KiCad 6
Other:
- net class Default removed
- board text added: "~{CS}"
- board text added: "~{MCS}"
- board text added: "~{MRD}"
- board text added: "~{MWR}"
- board text added: "~{RD}"
- board text added: "~{RES}"
- board text added: "~{WR}"
- board text removed: "~CS"
- board text removed: "~MCS"
- board text removed: "~MRD"
- board text removed: "~MWR"
- board text removed: "~RD"
- board text removed: "~RES"
- board text removed: "~WR"
