File: GB-BRK-M-XS/GB-BRK-M-XS.kicad_pcb (KiCad board)
At the start: 2 copper layers, 51.4 x 25 mm, 4 parts, among them J1 CONN_02X16, J2 Conn_GameBoy_Cartridge

Commit message: Adjust solder mask clearances, regenerate gerbers
Other:
- rule pad_to_mask_clearance: 0.2 -> 0
- rule solder_mask_min_width: 0.25 -> 0.2
Changed lines of the file:
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@@
     (pad_size 2.25 2.25)
     (pad_drill 2.25)
-    (pad_to_mask_clearance 0.2)
-    (solder_mask_min_width 0.25)
+    (pad_to_mask_clearance 0)
+    (solder_mask_min_width 0.2)
     (aux_axis_origin 100 100)
     (visible_elements FFFFFF7F)
     (pcbplotparams
-      (layerselection 0x010fc_80000001)
+      (layerselection 0x010fc_ffffffff)
       (usegerberextensions false)
       (usegerberattributes false)
       (usegerberadvancedattributes false)
-      (creategerberjobfile false)
+      (creategerberjobfile true)
       (excludeedgelayer false)
       (linewidth 0.100000)

Commit message: Set solder mask min width to 0, regenerate gerbers
Other:
- rule trace_min: 0.21 -> 0.2

Commit message: Rescue GB-BRK-M-XS and convert to KiCad 6
Connections:
- net ~CS renamed ~{CS}
- net ~RD renamed ~{RD}
- net ~RES renamed ~{RES}
- net ~WR renamed ~{WR}
Other:
- net class Default removed
- net class Power removed
