File: GB-CART32K-A/GB-CART32K-A.kicad_pcb (KiCad board)
At the start: 2 copper layers, 51.4 x 61 mm, 14 parts, among them J1 DNF, U1 SST39SF040

Commit message: Update GB-CART32K-A
Other:
- board text added: "32k-512k JEDEC 5V"
- board text added: "GB-CART32K-A v1.1 https://gekkio.fi"
- board text removed: "32k-512k x8 JEDEC 5V"
- board text removed: "GB-CART32K-A v1.0 https://gekkio.fi"
Changed lines of the file:
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@@
-(kicad_pcb (version 20171130) (host pcbnew 5.1.2-f72e74a~84~ubuntu19.04.1)
+(kicad_pcb (version 20171130) (host pcbnew 5.1.5-52549c5~84~ubuntu19.10.1)
   (general
     (thickness 1)
@@
   (title_block
     (title GB-CART32K-A)
-    (rev v1.0)
+    (rev v1.1)
     (company https://gekkio.fi)
   )
@@
   )
   (setup
-    (last_trace_width 0.6)
+    (last_trace_width 0.3)
     (user_trace_width 0.6)
     (trace_clearance 0.3)
@@
     (add_net /~ROM_WR)
     (add_net GND)
+    (add_net "Net-(J1-Pad2)")
+    (add_net "Net-(J1-Pad3)")
+    (add_net "Net-(J1-Pad30)")
+    (add_net "Net-(J1-Pad5)")
   )
   (module TestPoint:TestPoint_THTPad_D2.0mm_Drill1.0mm (layer F.Cu)
@@
     (pad "" np_thru_hole circle (at 0 0) (size 7.2 7.2) (drill 7.2) (layers *.Cu *.Mask))
   )
-  (gr_text "32k-512k x8\nJEDEC\n5V" (at 88.9 66) (layer F.SilkS)
+  (gr_text "32k-512k\nJEDEC\n5V" (at 88.9 66) (layer F.SilkS)
     (effects (font (size 1 1) (thickness 0.15)))
   )
@@
   (gr_arc (start 76.3 99.1) (end 75.4 99.1) (angle -90) (layer Edge.Cuts) (width 0.15))
   (gr_arc (start 123.7 99.1) (end 123.7 100) (angle -90) (layer Edge.Cuts) (width 0.15))
-  (gr_text "GB-CART32K-A v1.0\nhttps://gekkio.fi" (at 109.9 44.4) (layer F.SilkS)
+  (gr_text "GB-CART32K-A v1.1\nhttps://gekkio.fi" (at 109.9 44.4) (layer F.SilkS)
     (effects (font (size 1.2 1.2) (thickness 0.2)))
   )

Commit message: Upgrade most projects to KiCad 6
Connections:
- net /~RD renamed /~{RD}
- net /~ROM_CS renamed /~{ROM_CS}
- net /~ROM_WR renamed /~{ROM_WR}
Other:
- net class Default removed
- board text added: "A15/~{ROM_CS}"
- board text added: "~{RD}"
- board text added: "~{ROM_WR}"
- board text removed: "A15/~ROM_CS"
- board text removed: "~RD"
- board text removed: "~ROM_WR"
